File: pcb/nes-port-breadboard.kicad_pcb (KiCad board)
At the start: 2 copper layers, 38.1 x 38.1 mm, 2 parts, among them J1 Conn_01x07, J2 NES_Port_Male

Commit message: Rename nes-breadboard -> nes-port-breadboard
Parts:
- J2: footprint nes-breadboard:NES_Port_Male_Horizontal -> nes-port-breadboard:NES_Port_Male_Horizontal
Changed lines of the file:
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@@
     (add_net "Net-(J1-Pad7)")
   )
-  (module nes-breadboard:NES_Port_Male_Horizontal (layer F.Cu)
+  (module nes-port-breadboard:NES_Port_Male_Horizontal (layer F.Cu)
     (at 147.574 107.696)
     (fp_text reference J2 (at -11.2776 -14.0462) (layer F.SilkS)
@@
       (effects (font (size 1 1) (thickness 0.15)))
     )
+    (fp_line (start 1.8 -1.8) (end -1.8 -1.8) (layer F.CrtYd) (width 0.05))
+    (fp_line (start 1.8 17.05) (end 1.8 -1.8) (layer F.CrtYd) (width 0.05))
+    (fp_line (start -1.8 17.05) (end 1.8 17.05) (layer F.CrtYd) (width 0.05))
+    (fp_line (start -1.8 -1.8) (end -1.8 17.05) (layer F.CrtYd) (width 0.05))
+    (fp_line (start -1.33 -1.33) (end 0 -1.33) (layer F.SilkS) (width 0.12))
+    (fp_line (start -1.33 0) (end -1.33 -1.33) (layer F.SilkS) (width 0.12))
+    (fp_line (start -1.33 1.27) (end 1.33 1.27) (layer F.SilkS) (width 0.12))
+    (fp_line (start 1.33 1.27) (end 1.33 16.57) (layer F.SilkS) (width 0.12))
+    (fp_line (start -1.33 1.27) (end -1.33 16.57) (layer F.SilkS) (width 0.12))
+    (fp_line (start -1.33 16.57) (end 1.33 16.57) (layer F.SilkS) (width 0.12))
+    (fp_line (start -1.27 -0.635) (end -0.635 -1.27) (layer F.Fab) (width 0.1))
+    (fp_line (start -1.27 16.51) (end -1.27 -0.635) (layer F.Fab) (width 0.1))
+    (fp_line (start 1.27 16.51) (end -1.27 16.51) (layer F.Fab) (width 0.1))
+    (fp_line (start 1.27 -1.27) (end 1.27 16.51) (layer F.Fab) (width 0.1))
     (fp_line (start -0.635 -1.27) (end 1.27 -1.27) (layer F.Fab) (width 0.1))
-    (fp_line (start 1.27 -1.27) (end 1.27 16.51) (layer F.Fab) (width 0.1))
-    (fp_line (start 1.27 16.51) (end -1.27 16.51) (layer F.Fab) (width 0.1))
-    (fp_line (start -1.27 16.51) (end -1.27 -0.635) (layer F.Fab) (width 0.1))
-    (fp_line (start -1.27 -0.635) (end -0.635 -1.27) (layer F.Fab) (width 0.1))
-    (fp_line (start -1.33 16.57) (end 1.33 16.57) (layer F.SilkS) (width 0.12))
-    (fp_line (start -1.33 1.27) (end -1.33 16.57) (layer F.SilkS) (width 0.12))
-    (fp_line (start 1.33 1.27) (end 1.33 16.57) (layer F.SilkS) (width 0.12))
-    (fp_line (start -1.33 1.27) (end 1.33 1.27) (layer F.SilkS) (width 0.12))
-    (fp_line (start -1.33 0) (end -1.33 -1.33) (layer F.SilkS) (width 0.12))
-    (fp_line (start -1.33 -1.33) (end 0 -1.33) (layer F.SilkS) (width 0.12))
-    (fp_line (start -1.8 -1.8) (end -1.8 17.05) (layer F.CrtYd) (width 0.05))
-    (fp_line (start -1.8 17.05) (end 1.8 17.05) (layer F.CrtYd) (width 0.05))
-    (fp_line (start 1.8 17.05) (end 1.8 -1.8) (layer F.CrtYd) (width 0.05))
-    (fp_line (start 1.8 -1.8) (end -1.8 -1.8) (layer F.CrtYd) (width 0.05))
     (fp_text user %R (at 0 7.62 90) (layer F.Fab)
       (effects (font (size 1 1) (thickness 0.15)))
